Commit message: update multi-robot

File: d4nc3r_gz/urdf/d4nc3r_gz.xacro (robot description, xacro)
@@ -1,4 +1,5 @@
 <?xml version="1.0"?>
 <robot xmlns:xacro="http://www.ros.org/wiki/xacro" name="d4nc3r">
+  <xacro:property name="robot_namespace" value="/$(arg namespace)"/>
   <xacro:include filename="$(find d4nc3r_description)/urdf/d4nc3r.urdf.xacro"/>
    <xacro:if value="$(arg use_gazebo_ros_control)">
