Commit message: ok

File: d4nc3r_description/urdf/d4nc3r.urdf.xacro (robot description, xacro)
@@ -18,6 +18,4 @@
   <xacro:property name="second_base_yaml" value="$(arg yaml_config_dir)/second_base.yaml" />
   <xacro:property name="second_base_props" value="${xacro.load_yaml(second_base_yaml)}"/>
-  <xacro:property name="hardware_yaml" value="$(arg yaml_config_dir)/hardware.yaml" />
-  <xacro:property name="hardware_props" value="${xacro.load_yaml(hardware_yaml)}"/>
   <!-- Footprint link -->
   <xacro:footprint wheel_props="${wheel_props}" />
@@ -30,4 +28,10 @@
     <origin xyz="0 0 0.001" rpy="0 0 0" />
   </xacro:base>
+  <link name="dummy">
+   </link>
+  <joint name="dummy_joint" type="fixed">
+     <parent link="dummy"/>
+     <child link="base_link"/>
+   </joint>
   <!-- Joint to connect second_story with base_link -->
   <joint name="second_base_joint" type="fixed">
@@ -62,5 +66,4 @@
   <xacro:if value="$(arg use_real_ros_control)">
     <xacro:include filename="$(find ${package_name})/urdf/include/d4nc3r_control.urdf.xacro" />
-    <xacro:control hardware_props="${hardware_props}" />
   </xacro:if>
 </robot>

File: d4nc3r_description/urdf/include/d4nc3r_control.urdf.xacro (robot description, xacro)
@@ -8,13 +8,4 @@
     <!-- TODO(francocipollone): This xacro should be part of andino_control package instead.-->
     <ros2_control name="RealRobot" type="system">
-      <hardware>
-        <plugin>andino_base/DiffDriveAndino</plugin>
-        <param name="left_wheel_name">${hardware_props['left_wheel_name']}</param>
-        <param name="right_wheel_name">${hardware_props['right_wheel_name']}</param>
-        <param name="serial_device">${hardware_props['serial_device']}</param>
-        <param name="baud_rate">${hardware_props['baud_rate']}</param>
-        <param name="timeout">${hardware_props['timeout']}</param>
-        <param name="enc_ticks_per_rev">${hardware_props['enc_ticks_per_rev']}</param>
-      </hardware>
       <joint name="left_wheel_joint">
         <command_interface name="velocity">

Commit message: teste01

File: d4nc3r_description/urdf/d4nc3r.urdf.xacro (robot description, xacro)
@@ -9,5 +9,4 @@
   <xacro:property name="caster_wheel_props" value="${xacro.load_yaml(caster_wheel_yaml)}"/>
   <xacro:arg name="use_fixed_caster" default="True"/>
-  <xacro:arg name="use_real_ros_control" default="True"/>
   <xacro:property name="wheel_yaml" value="$(arg yaml_config_dir)/wheel.yaml" />
   <xacro:property name="wheel_props" value="${xacro.load_yaml(wheel_yaml)}"/>
@@ -28,10 +27,4 @@
     <origin xyz="0 0 0.001" rpy="0 0 0" />
   </xacro:base>
-  <link name="dummy">
-   </link>
-  <joint name="dummy_joint" type="fixed">
-     <parent link="dummy"/>
-     <child link="base_link"/>
-   </joint>
   <!-- Joint to connect second_story with base_link -->
   <joint name="second_base_joint" type="fixed">
@@ -48,10 +41,8 @@
   <xacro:wheel prefix="right" reflect="-1"
                       wheel_props="${wheel_props}"
-                      base_props="${base_props}" >
-  </xacro:wheel>
+                      base_props="${base_props}" />
   <xacro:wheel prefix="left" reflect="1"
                       wheel_props="${wheel_props}"
-                      base_props="${base_props}" >
-  </xacro:wheel>
+                      base_props="${base_props}" />
   <!-- Motors -->
   <xacro:motor prefix="right" reflect="-1"
@@ -63,7 +54,17 @@
                       base_props="${base_props}" >
   </xacro:motor>
-  <!-- ros2_control -->
-  <xacro:if value="$(arg use_real_ros_control)">
-    <xacro:include filename="$(find ${package_name})/urdf/include/d4nc3r_control.urdf.xacro" />
-  </xacro:if>
+  <!-- Odometria link -->
+  <link name="odom_link"/>
+  <joint name="odom_joint" type="fixed">
+    <parent link="base_link"/>
+    <child link="odom_link"/>
+    <origin xyz="0 0 0" rpy="0 0 3.1416"/>
+  </joint>
+  <!-- MPU link -->
+  <link name="mpu_link"/>
+  <joint name="mpu_joint" type="fixed">
+    <parent link="base_link"/>
+    <child link="mpu_link"/>
+    <origin xyz="-0.033 -0.010 0.02" rpy="0 0 3.1416"/>
+  </joint>
 </robot>

File: d4nc3r_description/urdf/include/common_macros.urdf.xacro (robot description, xacro)
@@ -132,10 +132,6 @@
                params="link_name:='base_link' base_prop mesh:='' scale:='' *origin ">
     <link name="${link_name}">
-    <xacro:cylinder_inertia m="${base_prop['base']['mass']}"
-                              r="${base_prop['base']['diameter']}"
-                              l="${base_prop['base']['height']}"
-                              o_xyz="0.0 0.0 0.0"
-                              o_rpy="${pi/2.0} 0.0 0.0" >
-    </xacro:cylinder_inertia>
+    <!-- Remover a inércia do link raiz -->
+    <!-- <xacro:cylinder_inertia ... /> -->
     <xacro:if value="${mesh != '' }" >
       <visual>
@@ -180,6 +176,12 @@
                params="wheel_props">
     <!-- Base-Footprint -->
-    <!-- base_footprint is a fictitious link(frame) that is on the ground right below base_link origin -->
-    <link name="base_footprint" />
+    <link name="base_footprint">
+      <!-- Adicionar a inércia aqui -->
+      <xacro:cylinder_inertia m="${wheel_props['mass']}"
+                              r="${wheel_props['radius']}"
+                              l="${wheel_props['length']}"
+                              o_xyz="0.0 0.0 0.0"
+                              o_rpy="${pi/2.0} 0.0 0.0" />
+    </link>
     <!-- Joint to connect base_footprint with base_link -->
     <joint name="base_footprint_joint" type="fixed">

Commit message: ok

File: d4nc3r_description/urdf/d4nc3r.urdf.xacro (robot description, xacro)
@@ -68,3 +68,22 @@
     <origin xyz="-0.033 -0.010 0.02" rpy="0 0 3.1416"/>
   </joint>
+    <ros2_control name="D4nc3rRealHardware" type="system">
+    <hardware>
+      <plugin>d4nc3r_control/D4nc3rHardwareInterface</plugin>
+      <param name="encoder_topic_name">/d4nc3r1/encoders</param>
+      <param name="ticks_per_wheel_revolution">8.0</param>
+      <param name="left_encoder_data_index">1</param>
+      <param name="right_encoder_data_index">0</param>
+    </hardware>
+    <joint name="left_wheel_joint"> <!-- No type attribute here - correct -->
+      <command_interface name="velocity"/>
+      <state_interface name="position"/>
+      <state_interface name="velocity"/>
+    </joint>
+    <joint name="right_wheel_joint"> <!-- No type attribute here - correct -->
+      <command_interface name="velocity"/>
+      <state_interface name="position"/>
+      <state_interface name="velocity"/>
+    </joint>
+  </ros2_control>
 </robot>

Commit message: fiz urdf

File: d4nc3r_description/urdf/d4nc3r.urdf.xacro (robot description, xacro)
@@ -66,5 +66,5 @@
     <parent link="base_link"/>
     <child link="mpu_link"/>
-    <origin xyz="-0.033 -0.010 0.02" rpy="0 0 3.1416"/>
+    <origin xyz="-0.033 -0.010 0.02" rpy="3.1416 0 0"/> <!-- Corrija a orientação aqui -->
   </joint>
     <ros2_control name="D4nc3rRealHardware" type="system">

Commit message: update_2

File: d4nc3r_description/urdf/d4nc3r.urdf.xacro (robot description, xacro)
@@ -2,6 +2,7 @@
 <robot xmlns:xacro="http://www.ros.org/wiki/xacro" name="d4nc3r">
   <xacro:property name="package_name" value="d4nc3r_description"/>
-  <xacro:property name="robot_name" value="d4nc3r"/>
-z
+  <xacro:property name="robot_name" value="d4nc3r"/> <!-- Used for mesh paths, should remain 'd4nc3r' -->
+  <xacro:arg name="frame_prefix_arg" default="0"/> <!-- Argument from launch file for prefixing -->
+  <xacro:property name="processed_prefix" value="$(arg frame_prefix_arg)_" /> <!-- Prefix with underscore otherwise -->
   <xacro:include filename="$(find ${package_name})/urdf/include/common_macros.urdf.xacro" />
   <xacro:include filename="$(find ${package_name})/urdf/include/d4nc3r_caster_macro.urdf.xacro" />
@@ -19,52 +20,60 @@
   <xacro:property name="second_base_props" value="${xacro.load_yaml(second_base_yaml)}"/>
   <!-- Footprint link -->
-  <xacro:footprint wheel_props="${wheel_props}" />
+  <xacro:footprint robot_prefix="${processed_prefix}"
+                   wheel_props="${wheel_props}" />
   <!-- Base link -->
-  <xacro:base link_name="base_link" base_prop="${base_props}" mesh="${base_props['base']['mesh']}" >
+  <xacro:base robot_prefix="${processed_prefix}"
+              link_name="base_link" base_prop="${base_props}" mesh="${base_props['base']['mesh']}" >
     <origin xyz="0 0 0" rpy="0 0 0" />
   </xacro:base>
   <!-- Second story link -->
-  <xacro:base link_name="second_base_link" base_prop="${second_base_props}" mesh="${second_base_props['base']['mesh']}" >
+  <xacro:base robot_prefix="${processed_prefix}"
+              link_name="second_base_link" base_prop="${second_base_props}" mesh="${second_base_props['base']['mesh']}" >
     <origin xyz="0 0 0.001" rpy="0 0 0" />
   </xacro:base>
   <!-- Joint to connect second_story with base_link -->
-  <joint name="second_base_joint" type="fixed">
-    <parent link="base_link"/>
-    <child link="second_base_link" />
+  <joint name="${processed_prefix}second_base_joint" type="fixed">
+    <parent link="${processed_prefix}base_link"/>
+    <child link="${processed_prefix}second_base_link" />
     <origin xyz="0 0 0" rpy="0 0 0" />
   </joint>
   <!-- Caster Wheel -->
-  <xacro:caster_wheel reflect="-1"
+  <xacro:caster_wheel robot_prefix="${processed_prefix}"
+                      reflect="-1"
                       use_fixed="$(arg use_fixed_caster)"
                       wheel_props="${caster_wheel_props}">
   </xacro:caster_wheel>
   <!-- Wheels -->
-  <xacro:wheel prefix="right" reflect="-1"
+  <xacro:wheel robot_prefix="${processed_prefix}"
+               prefix="right" reflect="-1"
                       wheel_props="${wheel_props}"
                       base_props="${base_props}" />
-  <xacro:wheel prefix="left" reflect="1"
+  <xacro:wheel robot_prefix="${processed_prefix}"
+               prefix="left" reflect="1"
                       wheel_props="${wheel_props}"
                       base_props="${base_props}" />
   <!-- Motors -->
-  <xacro:motor prefix="right" reflect="-1"
+  <xacro:motor robot_prefix="${processed_prefix}"
+               prefix="right" reflect="-1"
                       motor_props="${motor_props}"
                       base_props="${base_props}" >
   </xacro:motor>
-  <xacro:motor prefix="left" reflect="1"
+  <xacro:motor robot_prefix="${processed_prefix}"
+               prefix="left" reflect="1"
                       motor_props="${motor_props}"
                       base_props="${base_props}" >
   </xacro:motor>
   <!-- Odometria link -->
-  <link name="odom_link"/>
-  <joint name="odom_joint" type="fixed">
-    <parent link="base_link"/>
-    <child link="odom_link"/>
+  <link name="${processed_prefix}odom_link"/>
+  <joint name="${processed_prefix}odom_joint" type="fixed">
+    <parent link="${processed_prefix}base_link"/>
+    <child link="${processed_prefix}odom_link"/>
     <origin xyz="0 0 0" rpy="0 0 3.1416"/>
   </joint>
   <!-- MPU link -->
-  <link name="mpu_link"/>
-  <joint name="mpu_joint" type="fixed">
-    <parent link="base_link"/>
-    <child link="mpu_link"/>
+  <link name="${processed_prefix}mpu_link"/>
+  <joint name="${processed_prefix}mpu_joint" type="fixed">
+    <parent link="${processed_prefix}base_link"/>
+    <child link="${processed_prefix}mpu_link"/>
     <origin xyz="-0.033 -0.010 0.02" rpy="3.1416 0 0"/> <!-- Corrija a orientação aqui -->
   </joint>
@@ -77,10 +86,10 @@
       <param name="right_encoder_data_index">0</param>
     </hardware>
-    <joint name="left_wheel_joint"> <!-- No type attribute here - correct -->
+    <joint name="${processed_prefix}left_wheel_joint"> <!-- No type attribute here - correct -->
       <command_interface name="velocity"/>
       <state_interface name="position"/>
       <state_interface name="velocity"/>
     </joint>
-    <joint name="right_wheel_joint"> <!-- No type attribute here - correct -->
+    <joint name="${processed_prefix}right_wheel_joint"> <!-- No type attribute here - correct -->
       <command_interface name="velocity"/>
       <state_interface name="position"/>

File: d4nc3r_description/urdf/include/common_macros.urdf.xacro (robot description, xacro)
@@ -11,5 +11,5 @@
 -->
   <xacro:macro name="wheel"
-               params="prefix reflect wheel_props base_props ">
+               params="robot_prefix prefix reflect wheel_props base_props ">
   <xacro:property name="pos_x_joint"
      value="${(base_props['base']['x_size']/2) - wheel_props['x_offset']}"/>
@@ -17,5 +17,5 @@
     value="${(base_props['base']['y_size']/2) + wheel_props['y_offset'] + (wheel_props['length']/2)}"/>
   <xacro:property name="pos_z_joint" value="${wheel_props['z_offset']}"/>
-    <link name="${prefix}_wheel">
+    <link name="${robot_prefix}${prefix}_wheel">
     <xacro:if value="${wheel_props['mesh'] != '' }" >
       <visual>
@@ -54,8 +54,8 @@
       </xacro:cylinder_inertia>
     </link>
-    <joint name="${prefix}_wheel_joint" type="continuous">
+    <joint name="${robot_prefix}${prefix}_wheel_joint" type="continuous">
       <axis xyz="0 1 0" rpy="0 0 0" />
-      <parent link="base_link"/>
-      <child link="${prefix}_wheel"/>
+      <parent link="${robot_prefix}base_link"/> <!-- Assuming base_link is the standard name for the main base -->
+      <child link="${robot_prefix}${prefix}_wheel"/>
       <origin xyz="${pos_x_joint} ${reflect* pos_y_joint} ${pos_z_joint}" rpy="0 0 0"/>
       <dynamics damping="0.01" friction="0.0"/>
@@ -72,5 +72,5 @@
 -->
   <xacro:macro name="motor"
-               params="prefix reflect motor_props base_props ">
+               params="robot_prefix prefix reflect motor_props base_props ">
   <xacro:property name="pos_x_joint"
      value="${(base_props['base']['x_size']/2) - motor_props['x_offset']}"/>
@@ -78,5 +78,5 @@
     value="${(base_props['base']['y_size']/2) + motor_props['y_offset'] + (motor_props['y_size']/2)}"/>
   <xacro:property name="pos_z_joint" value="${motor_props['z_offset']}"/>
-    <link name="${prefix}_motor">
+    <link name="${robot_prefix}${prefix}_motor">
     <xacro:if value="${motor_props['mesh'] != '' }" >
       <visual>
@@ -114,7 +114,7 @@
       </xacro:box_inertia>
     </link>
-    <joint name="${prefix}_motor_joint" type="fixed">
-      <parent link="base_link"/>
-      <child link="${prefix}_motor"/>
+    <joint name="${robot_prefix}${prefix}_motor_joint" type="fixed">
+      <parent link="${robot_prefix}base_link"/> <!-- Assuming base_link is the standard name for the main base -->
+      <child link="${robot_prefix}${prefix}_motor"/>
       <origin xyz="${pos_x_joint} ${reflect* pos_y_joint} ${pos_z_joint}" rpy="0 ${-pi/2.0*(reflect - 1)} 0"/>
       <axis xyz="0 1 0" rpy="0 0 0" />
@@ -130,6 +130,6 @@
 -->
   <xacro:macro name="base"
-               params="link_name:='base_link' base_prop mesh:='' scale:='' *origin ">
-    <link name="${link_name}">
+               params="robot_prefix link_name:='base_link' base_prop mesh:='' scale:='' *origin ">
+    <link name="${robot_prefix}${link_name}">
     <!-- Remover a inércia do link raiz -->
     <!-- <xacro:cylinder_inertia ... /> -->
@@ -174,7 +174,7 @@
 -->
   <xacro:macro name="footprint"
-               params="wheel_props">
+               params="robot_prefix wheel_props">
     <!-- Base-Footprint -->
-    <link name="base_footprint">
+    <link name="${robot_prefix}base_footprint">
       <!-- Adicionar a inércia aqui -->
       <xacro:cylinder_inertia m="${wheel_props['mass']}"
@@ -185,7 +185,7 @@
     </link>
     <!-- Joint to connect base_footprint with base_link -->
-    <joint name="base_footprint_joint" type="fixed">
-      <parent link="base_link"/>
-      <child link="base_footprint" />
+    <joint name="${robot_prefix}base_footprint_joint" type="fixed">
+      <parent link="${robot_prefix}base_link"/> <!-- Assuming base_link is the standard name for the main base -->
+      <child link="${robot_prefix}base_footprint" />
       <origin xyz="0 0 ${-(wheel_props['radius'] - wheel_props['z_offset'])}" rpy="0 0 0" />
     </joint>

File: d4nc3r_description/urdf/include/d4nc3r_caster_macro.urdf.xacro (robot description, xacro)
@@ -16,6 +16,6 @@
 <!-- Caster wheel link & joint macro -->
   <xacro:macro name="caster_wheel"
-                params="reflect use_fixed wheel_props locationright:=${0} scale:=''">
-    <link name="caster_base_link">
+                params="robot_prefix reflect use_fixed wheel_props locationright:=${0} scale:=''">
+    <link name="${robot_prefix}caster_base_link">
       <xacro:box_inertia  m="${wheel_props['base']['mass']}"
                           x="${wheel_props['base']['size']['x']}"
@@ -54,14 +54,14 @@
       </collision>
     </link>
-    <joint name="caster_base_joint" type="fixed">
+    <joint name="${robot_prefix}caster_base_joint" type="fixed">
       <origin xyz="${wheel_props['base']['dx']} ${-wheel_props['base']['dy'] * locationright} ${wheel_props['base']['dz']}"
               rpy="0 0 0" />
-      <parent link="base_link" />
-      <child link="caster_base_link" />
+      <parent link="${robot_prefix}base_link" />
+      <child link="${robot_prefix}caster_base_link" />
       <axis xyz="0 0 1" />
       <dynamics damping="0.01" friction="0.0"/>
     </joint>
     <!-- caster hub -->
-    <link name="caster_rotation_link">
+    <link name="${robot_prefix}caster_rotation_link">
       <xacro:box_inertia  m="${wheel_props['hub']['mass']}"
                           x="${wheel_props['hub']['size']['x']}"
@@ -101,9 +101,9 @@
     </link>
     <xacro:if value="${use_fixed}">
-      <joint name="caster_rotation_joint" type="fixed">
+      <joint name="${robot_prefix}caster_rotation_joint" type="fixed">
         <origin xyz="${wheel_props['hub']['dx']} ${-wheel_props['hub']['dy'] * locationright} ${wheel_props['hub']['dz']}"
                 rpy="0 0 0" />
-        <parent link="base_link" />
-        <child link="caster_rotation_link" />
+        <parent link="${robot_prefix}base_link" /> <!-- As per original structure, parented to base_link -->
+        <child link="${robot_prefix}caster_rotation_link" />
         <axis xyz="0 0 1" />
         <dynamics damping="0.01" friction="0.0"/>
@@ -111,9 +111,9 @@
     </xacro:if>
     <xacro:unless value="${use_fixed}">
-      <joint name="caster_rotation_joint" type="continuous">
+      <joint name="${robot_prefix}caster_rotation_joint" type="continuous">
         <origin xyz="${wheel_props['hub']['dx']} ${-wheel_props['hub']['dy'] * locationright} ${wheel_props['hub']['dz']}"
                 rpy="0 0 0" />
-        <parent link="base_link" />
-        <child link="caster_rotation_link" />
+        <parent link="${robot_prefix}base_link" /> <!-- As per original structure, parented to base_link -->
+        <child link="${robot_prefix}caster_rotation_link" />
         <axis xyz="0 0 1" />
         <dynamics damping="0.01" friction="0.0"/>
@@ -121,5 +121,5 @@
     </xacro:unless>
     <!-- caster wheel -->
-    <link name="caster_wheel_link">
+    <link name="${robot_prefix}caster_wheel_link">
       <xacro:cylinder_inertia m="${wheel_props['wheel']['mass']}"
                               r="${wheel_props['wheel']['radius']}"
@@ -157,18 +157,18 @@
     </link>
     <xacro:if value="${use_fixed}">
-      <joint name="caster_wheel_joint" type="fixed">
+      <joint name="${robot_prefix}caster_wheel_joint" type="fixed">
         <origin xyz="${wheel_props['wheel']['dx']} ${-wheel_props['wheel']['dy'] * locationright} ${wheel_props['wheel']['dz']}"
                 rpy="0 0 0" />
-        <parent link="caster_rotation_link" />
-        <child link="caster_wheel_link" />
+        <parent link="${robot_prefix}caster_rotation_link" />
+        <child link="${robot_prefix}caster_wheel_link" />
         <axis xyz="0 1 0" />
       </joint>
     </xacro:if>
     <xacro:unless value="${use_fixed}">
-      <joint name="caster_wheel_joint" type="continuous">
+      <joint name="${robot_prefix}caster_wheel_joint" type="continuous">
         <origin xyz="${wheel_props['wheel']['dx']} ${-wheel_props['wheel']['dy'] * locationright} ${wheel_props['wheel']['dz']}"
                 rpy="0 0 0" />
-        <parent link="caster_rotation_link" />
-        <child link="caster_wheel_link" />
+        <parent link="${robot_prefix}caster_rotation_link" />
+        <child link="${robot_prefix}caster_wheel_link" />
         <axis xyz="0 1 0" />
       </joint>
